Commit message: plane constant velocity tracking (0.07) without depth_camera and height_map

File: gym/assets/urdf/neuroant.urdf (robot description, URDF)
Before this commit: robot nueroant, 19 links, 18 joints
Links:
- link l1_bc: geometry visual mesh filename=../meshes/l1_bc.STL
- link l1_cf: geometry visual mesh filename=../meshes/l1_cf.STL
- link l2_bc: geometry visual mesh filename=../meshes/l2_bc.STL
- link l2_cf: geometry visual mesh filename=../meshes/l2_cf.STL
- link l3_bc: geometry visual mesh filename=../meshes/l3_bc.STL
- link l3_cf: geometry visual mesh filename=../meshes/l3_cf.STL
- link r1_bc: geometry visual mesh filename=../meshes/r1_bc.STL
- link r1_cf: geometry visual mesh filename=../meshes/r1_cf.STL
- link r2_bc: geometry visual mesh filename=../meshes/r2_bc.STL
- link r2_cf: geometry visual mesh filename=../meshes/r2_cf.STL
- link r3_bc: geometry visual mesh filename=../meshes/r3_bc.STL
- link r3_cf: geometry visual mesh filename=../meshes/r3_cf.STL
Joints:
- joint l1_bc: limit lower=-3.14 upper=3.14 effort=4.2 velocity=1000 -> lower=-0.53 upper=0.53 effort=30 velocity=28.6
- joint l1_cf: limit lower=-3.14 upper=3.14 effort=4.2 velocity=1000 -> lower=-0.53 upper=0.53 effort=30 velocity=28.6
- joint l1_ft: limit lower=-3.14 upper=3.14 effort=4.2 velocity=1000 -> lower=-0.53 upper=0.53 effort=30 velocity=28.6
- joint l2_bc: limit lower=-3.14 upper=3.14 effort=4.2 velocity=1000 -> lower=-0.53 upper=0.53 effort=30 velocity=28.6
- joint l2_cf: limit lower=-3.14 upper=3.14 effort=4.2 velocity=1000 -> lower=-0.53 upper=0.53 effort=30 velocity=28.6
- joint l2_ft: limit lower=-3.14 upper=3.14 effort=4.2 velocity=1000 -> lower=-0.53 upper=0.53 effort=30 velocity=28.6
- joint l3_bc: limit lower=-3.14 upper=3.14 effort=4.2 velocity=1000 -> lower=-0.53 upper=0.53 effort=30 velocity=28.6
- joint l3_cf: limit lower=-3.14 upper=3.14 effort=4.2 velocity=1000 -> lower=-0.53 upper=0.53 effort=30 velocity=28.6
- joint l3_ft: limit lower=-3.14 upper=3.14 effort=4.2 velocity=1000 -> lower=-0.53 upper=0.53 effort=30 velocity=28.6
- joint r1_bc: limit lower=-3.14 upper=3.14 effort=4.2 velocity=1000 -> lower=-0.53 upper=0.53 effort=30 velocity=28.6
- joint r1_cf: limit lower=-3.14 upper=3.14 effort=4.2 velocity=1000 -> lower=-0.53 upper=0.53 effort=30 velocity=28.6
- joint r1_ft: limit lower=-3.14 upper=3.14 effort=4.2 velocity=1000 -> lower=-0.53 upper=0.53 effort=30 velocity=28.6
- joint r2_bc: limit lower=-3.14 upper=3.14 effort=4.2 velocity=1000 -> lower=-0.53 upper=0.53 effort=30 velocity=28.6
- joint r2_cf: limit lower=-3.14 upper=3.14 effort=4.2 velocity=1000 -> lower=-0.53 upper=0.53 effort=30 velocity=28.6
- joint r2_ft: limit lower=-3.14 upper=3.14 effort=4.2 velocity=1000 -> lower=-0.53 upper=0.53 effort=30 velocity=28.6
- joint r3_bc: limit lower=-3.14 upper=3.14 effort=4.2 velocity=1000 -> lower=-0.53 upper=0.53 effort=30 velocity=28.6
- joint r3_cf: limit lower=-3.14 upper=3.14 effort=4.2 velocity=1000 -> lower=-0.53 upper=0.53 effort=30 velocity=28.6
- joint r3_ft: limit lower=-3.14 upper=3.14 effort=4.2 velocity=1000 -> lower=-0.53 upper=0.53 effort=30 velocity=28.6

Commit message: can run on curriculum level1 terrain

File: gym/assets/urdf/neuroant.urdf (robot description, URDF)
Before this commit: robot nueroant, 19 links, 18 joints
Links:
- added link l1_foot_tip, mass 0.06; collision sphere radius=0.008; visual sphere radius=0.008
- added link l2_foot_tip, mass 0.06; collision sphere radius=0.008; visual sphere radius=0.008
- added link l3_foot_tip, mass 0.06; collision sphere radius=0.008; visual sphere radius=0.008
- added link r1_foot_tip, mass 0.06; collision sphere radius=0.008; visual sphere radius=0.008
- added link r2_foot_tip, mass 0.06; collision sphere radius=0.008; visual sphere radius=0.008
- added link r3_foot_tip, mass 0.06; collision sphere radius=0.008; visual sphere radius=0.008
- link base_link: geometry collision box size=0.14 0.4 0.1; visual mesh filename=../meshes/base_link.STL
- link l1_bc: geometry collision box size=0.05 0.03 0.045; visual mesh filename=../meshes/l1_bc.STL
- link l1_ft: geometry collision box size=0.02 0.02 0.122; visual mesh filename=../meshes/l1_ft.STL
- link l2_bc: geometry collision box size=0.05 0.03 0.045; visual mesh filename=../meshes/l2_bc.STL
- link l2_ft: geometry collision box size=0.02 0.02 0.122; visual mesh filename=../meshes/l2_ft.STL
- link l3_bc: geometry collision box size=0.05 0.03 0.045; visual mesh filename=../meshes/l3_bc.STL
- link l3_ft: geometry collision box size=0.02 0.02 0.122; visual mesh filename=../meshes/l3_ft.STL
- link r1_bc: geometry collision box size=0.05 0.03 0.045; visual mesh filename=../meshes/r1_bc.STL
- link r1_ft: geometry collision box size=0.02 0.02 0.122; visual mesh filename=../meshes/r1_ft.STL
- link r2_bc: geometry collision box size=0.05 0.03 0.045; visual mesh filename=../meshes/r2_bc.STL
- link r2_ft: geometry collision box size=0.02 0.02 0.122; visual mesh filename=../meshes/r2_ft.STL
- link r3_bc: geometry collision box size=0.05 0.03 0.045; visual mesh filename=../meshes/r3_bc.STL
- link r3_ft: geometry collision box size=0.02 0.02 0.122; visual mesh filename=../meshes/r3_ft.STL
Joints:
- added joint l1_foot_joint: type fixed, parent l1_ft, child l1_foot_tip, origin xyz=-0.0337 -0.127 0 rpy=0 0 0
- added joint l2_foot_joint: type fixed, parent l2_ft, child l2_foot_tip, origin xyz=-0.0337 -0.127 0 rpy=0 0 0
- added joint l3_foot_joint: type fixed, parent l3_ft, child l3_foot_tip, origin xyz=-0.0337 -0.127 0 rpy=0 0 0
- added joint r1_foot_joint: type fixed, parent r1_ft, child r1_foot_tip, origin xyz=-0.0337 0.127 0 rpy=0 0 0
- added joint r2_foot_joint: type fixed, parent r2_ft, child r2_foot_tip, origin xyz=-0.0337 0.127 0 rpy=0 0 0
- added joint r3_foot_joint: type fixed, parent r3_ft, child r3_foot_tip, origin xyz=-0.0337 0.127 0 rpy=0 0 0
- joint l1_bc: limit lower=-0.53 upper=0.53 effort=30 velocity=28.6 -> lower=-0.7854 upper=0.7854 effort=20 velocity=20.0
- joint l1_cf: limit lower=-0.53 upper=0.53 effort=30 velocity=28.6 -> lower=-0.7854 upper=0.7854 effort=20 velocity=20.0
- joint l1_ft: limit lower=-0.53 upper=0.53 effort=30 velocity=28.6 -> lower=0.000 upper=0.7854 effort=20 velocity=20.0
- joint l2_bc: limit lower=-0.53 upper=0.53 effort=30 velocity=28.6 -> lower=-0.7854 upper=0.7854 effort=20 velocity=20.0
- joint l2_cf: limit lower=-0.53 upper=0.53 effort=30 velocity=28.6 -> lower=-0.7854 upper=0.7854 effort=20 velocity=20.0
- joint l2_ft: limit lower=-0.53 upper=0.53 effort=30 velocity=28.6 -> lower=0.000 upper=0.7854 effort=20 velocity=20.0
- joint l3_bc: limit lower=-0.53 upper=0.53 effort=30 velocity=28.6 -> lower=-0.7854 upper=0.7854 effort=20 velocity=20.0
- joint l3_cf: limit lower=-0.53 upper=0.53 effort=30 velocity=28.6 -> lower=-0.7854 upper=0.7854 effort=20 velocity=20.0
- joint l3_ft: limit lower=-0.53 upper=0.53 effort=30 velocity=28.6 -> lower=0.000 upper=0.7854 effort=20 velocity=20.0
- joint r1_bc: limit lower=-0.53 upper=0.53 effort=30 velocity=28.6 -> lower=-0.7854 upper=0.7854 effort=20 velocity=20.0
- joint r1_cf: limit lower=-0.53 upper=0.53 effort=30 velocity=28.6 -> lower=-0.7854 upper=0.7854 effort=20 velocity=20.0
- joint r1_ft: limit lower=-0.53 upper=0.53 effort=30 velocity=28.6 -> lower=-0.7854 upper=0 effort=20 velocity=20.0
- joint r2_bc: limit lower=-0.53 upper=0.53 effort=30 velocity=28.6 -> lower=-0.7854 upper=0.7854 effort=20 velocity=20.0
- joint r2_cf: limit lower=-0.53 upper=0.53 effort=30 velocity=28.6 -> lower=-0.7854 upper=0.7854 effort=20 velocity=20.0
- joint r2_ft: limit lower=-0.53 upper=0.53 effort=30 velocity=28.6 -> lower=-0.7854 upper=0 effort=20 velocity=20.0
- joint r3_bc: limit lower=-0.53 upper=0.53 effort=30 velocity=28.6 -> lower=-0.7854 upper=0.7854 effort=20 velocity=20.0
- joint r3_cf: limit lower=-0.53 upper=0.53 effort=30 velocity=28.6 -> lower=-0.7854 upper=0.7854 effort=20 velocity=20.0
- joint r3_ft: axis 0 1.9702E-05 1 -> 0 0 1; limit lower=-0.53 upper=0.53 effort=30 velocity=28.6 -> lower=-0.7854 upper=0 effort=20 velocity=20.0; origin xyz=0.064248 0 0 rpy=1.9702E-05 0 0.85317 -> xyz=0.0642484706341889 0 -4.06229553796666E-05 rpy=0 0 0.858119138737752

Commit message: average terrain levels 3

File: gym/assets/urdf/neuroant.urdf (robot description, URDF)
Before this commit: robot nueroant, 25 links, 24 joints
Joints:
- joint l1_bc: limit lower=-0.7854 upper=0.7854 effort=20 velocity=20.0 -> lower=-0.7854 upper=0.7854 effort=20 velocity=13.0
- joint l1_cf: limit lower=-0.7854 upper=0.7854 effort=20 velocity=20.0 -> lower=-0.7854 upper=0.7854 effort=20 velocity=13.0
- joint l1_ft: limit lower=0.000 upper=0.7854 effort=20 velocity=20.0 -> lower=0.000 upper=0.7854 effort=20 velocity=13.0
- joint l2_bc: limit lower=-0.7854 upper=0.7854 effort=20 velocity=20.0 -> lower=-0.7854 upper=0.7854 effort=20 velocity=13.0
- joint l2_cf: limit lower=-0.7854 upper=0.7854 effort=20 velocity=20.0 -> lower=-0.7854 upper=0.7854 effort=20 velocity=13.0
- joint l2_ft: limit lower=0.000 upper=0.7854 effort=20 velocity=20.0 -> lower=0.000 upper=0.7854 effort=20 velocity=13.0
- joint l3_bc: limit lower=-0.7854 upper=0.7854 effort=20 velocity=20.0 -> lower=-0.7854 upper=0.7854 effort=20 velocity=13.0
- joint l3_cf: limit lower=-0.7854 upper=0.7854 effort=20 velocity=20.0 -> lower=-0.7854 upper=0.7854 effort=20 velocity=13.0
- joint l3_ft: limit lower=0.000 upper=0.7854 effort=20 velocity=20.0 -> lower=0.000 upper=0.7854 effort=20 velocity=13.0
- joint r1_bc: limit lower=-0.7854 upper=0.7854 effort=20 velocity=20.0 -> lower=-0.7854 upper=0.7854 effort=20 velocity=13.0
- joint r1_cf: limit lower=-0.7854 upper=0.7854 effort=20 velocity=20.0 -> lower=-0.7854 upper=0.7854 effort=20 velocity=13.0
- joint r1_ft: limit lower=-0.7854 upper=0 effort=20 velocity=20.0 -> lower=-0.7854 upper=0 effort=20 velocity=13.0
- joint r2_bc: limit lower=-0.7854 upper=0.7854 effort=20 velocity=20.0 -> lower=-0.7854 upper=0.7854 effort=20 velocity=13.0
- joint r2_cf: limit lower=-0.7854 upper=0.7854 effort=20 velocity=20.0 -> lower=-0.7854 upper=0.7854 effort=20 velocity=13.0
- joint r2_ft: limit lower=-0.7854 upper=0 effort=20 velocity=20.0 -> lower=-0.7854 upper=0 effort=20 velocity=13.0
- joint r3_bc: limit lower=-0.7854 upper=0.7854 effort=20 velocity=20.0 -> lower=-0.7854 upper=0.7854 effort=20 velocity=13.0
- joint r3_cf: limit lower=-0.7854 upper=0.7854 effort=20 velocity=20.0 -> lower=-0.7854 upper=0.7854 effort=20 velocity=13.0
- joint r3_ft: limit lower=-0.7854 upper=0 effort=20 velocity=20.0 -> lower=-0.7854 upper=0 effort=20 velocity=13.0

Commit message: add camera

File: gym/assets/urdf/neuroant.urdf (robot description, URDF)
Before this commit: robot nueroant, 25 links, 24 joints
Joints:
- joint l1_bc: limit lower=-0.7854 upper=0.7854 effort=20 velocity=13.0 -> lower=-0.7854 upper=0.7854 effort=20 velocity=10.0
- joint l1_cf: limit lower=-0.7854 upper=0.7854 effort=20 velocity=13.0 -> lower=-0.7854 upper=0.7854 effort=20 velocity=10.0
- joint l1_ft: limit lower=0.000 upper=0.7854 effort=20 velocity=13.0 -> lower=0.000 upper=0.7854 effort=20 velocity=10.0
- joint l2_bc: limit lower=-0.7854 upper=0.7854 effort=20 velocity=13.0 -> lower=-0.7854 upper=0.7854 effort=20 velocity=10.0
- joint l2_cf: limit lower=-0.7854 upper=0.7854 effort=20 velocity=13.0 -> lower=-0.7854 upper=0.7854 effort=20 velocity=10.0
- joint l2_ft: limit lower=0.000 upper=0.7854 effort=20 velocity=13.0 -> lower=0.000 upper=0.7854 effort=20 velocity=10.0
- joint l3_bc: limit lower=-0.7854 upper=0.7854 effort=20 velocity=13.0 -> lower=-0.7854 upper=0.7854 effort=20 velocity=10.0
- joint l3_cf: limit lower=-0.7854 upper=0.7854 effort=20 velocity=13.0 -> lower=-0.7854 upper=0.7854 effort=20 velocity=10.0
- joint l3_ft: limit lower=0.000 upper=0.7854 effort=20 velocity=13.0 -> lower=0.000 upper=0.7854 effort=20 velocity=10.0
- joint r1_bc: limit lower=-0.7854 upper=0.7854 effort=20 velocity=13.0 -> lower=-0.7854 upper=0.7854 effort=20 velocity=10.0
- joint r1_cf: limit lower=-0.7854 upper=0.7854 effort=20 velocity=13.0 -> lower=-0.7854 upper=0.7854 effort=20 velocity=10.0
- joint r1_ft: limit lower=-0.7854 upper=0 effort=20 velocity=13.0 -> lower=-0.7854 upper=0 effort=20 velocity=10.0
- joint r2_bc: limit lower=-0.7854 upper=0.7854 effort=20 velocity=13.0 -> lower=-0.7854 upper=0.7854 effort=20 velocity=10.0
- joint r2_cf: limit lower=-0.7854 upper=0.7854 effort=20 velocity=13.0 -> lower=-0.7854 upper=0.7854 effort=20 velocity=10.0
- joint r2_ft: limit lower=-0.7854 upper=0 effort=20 velocity=13.0 -> lower=-0.7854 upper=0 effort=20 velocity=10.0
- joint r3_bc: limit lower=-0.7854 upper=0.7854 effort=20 velocity=13.0 -> lower=-0.7854 upper=0.7854 effort=20 velocity=10.0
- joint r3_cf: limit lower=-0.7854 upper=0.7854 effort=20 velocity=13.0 -> lower=-0.7854 upper=0.7854 effort=20 velocity=10.0
- joint r3_ft: limit lower=-0.7854 upper=0 effort=20 velocity=13.0 -> lower=-0.7854 upper=0 effort=20 velocity=10.0
